File: recruitment.kicad_sch (KiCad schematic)
At the start: 18 parts

Commit message: check transistor, TODO: R values and multiplier supply
Connections:
- net GND: now also Q?.3 (E); no longer Q?.2 (C)
- net at Comparator.2 (-), R1.2, R2.1: now also Q?.2 (C); no longer Q?.3 (E)
Other:
- moved on the sheet: Q?, R1, R?
Changed lines of the file:
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@@
   (junction (at 160.02 129.54) (diameter 0) (color 0 0 0 0)
   )
-  (junction (at 118.11 109.22) (diameter 0) (color 0 0 0 0)
-  )
-  (junction (at 172.72 109.22) (diameter 0) (color 0 0 0 0)
+  (junction (at 118.11 107.95) (diameter 0) (color 0 0 0 0)
   )
   (junction (at 118.11 83.82) (diameter 0) (color 0 0 0 0)
   )
-  (junction (at 172.72 129.54) (diameter 0) (color 0 0 0 0)
-  )
   (junction (at 144.78 85.09) (diameter 0) (color 0 0 0 0)
   )
+  (junction (at 170.18 107.95) (diameter 0) (color 0 0 0 0)
+  )
   (junction (at 148.59 54.61) (diameter 0) (color 0 0 0 0)
   )
@@
   (junction (at 160.02 137.16) (diameter 0) (color 0 0 0 0)
   )
+  (junction (at 181.61 129.54) (diameter 0) (color 0 0 0 0)
+  )
   (junction (at 140.97 85.09) (diameter 0) (color 0 0 0 0)
   )
   (junction (at 135.89 69.85) (diameter 0) (color 0 0 0 0)
   )
-  (junction (at 160.02 109.22) (diameter 0) (color 0 0 0 0)
-  )
-  (junction (at 193.04 124.46) (diameter 0) (color 0 0 0 0)
-  )
-  (wire (pts (xy 180.34 124.46) (xy 193.04 124.46))
-    (stroke (width 0) (type default) (color 0 0 0 0))
-  )
-  (wire (pts (xy 118.11 109.22) (xy 118.11 134.62))
-    (stroke (width 0) (type default) (color 0 0 0 0))
-  )
-  (wire (pts (xy 160.02 109.22) (xy 172.72 109.22))
-    (stroke (width 0) (type default) (color 0 0 0 0))
-  )
-  (wire (pts (xy 193.04 132.08) (xy 193.04 124.46))
+  (junction (at 160.02 107.95) (diameter 0) (color 0 0 0 0)
+  )
+  (junction (at 193.04 120.65) (diameter 0) (color 0 0 0 0)
+  )
+  (wire (pts (xy 181.61 129.54) (xy 199.39 129.54))
+    (stroke (width 0) (type default) (color 0 0 0 0))
+  )
+  (wire (pts (xy 181.61 120.65) (xy 193.04 120.65))
+    (stroke (width 0) (type default) (color 0 0 0 0))
+  )
+  (wire (pts (xy 118.11 100.33) (xy 118.11 107.95))
+    (stroke (width 0) (type default) (color 0 0 0 0))
+  )
+  (wire (pts (xy 160.02 107.95) (xy 170.18 107.95))
+    (stroke (width 0) (type default) (color 0 0 0 0))
+  )
+  (wire (pts (xy 193.04 132.08) (xy 193.04 120.65))
     (stroke (width 0) (type default) (color 0 0 0 0))
   )
@@
     (stroke (width 0) (type default) (color 0 0 0 0))
   )
-  (wire (pts (xy 172.72 107.95) (xy 172.72 109.22))
-    (stroke (width 0) (type default) (color 0 0 0 0))
-  )
   (wire (pts (xy 140.97 85.09) (xy 144.78 85.09))
     (stroke (width 0) (type default) (color 0 0 0 0))
@@
     (stroke (width 0) (type default) (color 0 0 0 0))
   )
+  (wire (pts (xy 118.11 107.95) (xy 118.11 134.62))
+    (stroke (width 0) (type default) (color 0 0 0 0))
+  )
   (wire (pts (xy 144.78 85.09) (xy 154.94 85.09))
     (stroke (width 0) (type default) (color 0 0 0 0))
@@
     (stroke (width 0) (type default) (color 0 0 0 0))
   )
+  (wire (pts (xy 181.61 115.57) (xy 181.61 129.54))
+    (stroke (width 0) (type default) (color 0 0 0 0))
+  )
   (wire (pts (xy 104.14 57.15) (xy 120.65 57.15))
     (stroke (width 0) (type default) (color 0 0 0 0))
@@
     (stroke (width 0) (type default) (color 0 0 0 0))
   )
-  (wire (pts (xy 172.72 109.22) (xy 172.72 119.38))
+  (wire (pts (xy 173.99 115.57) (xy 181.61 115.57))
     (stroke (width 0) (type default) (color 0 0 0 0))
   )
@@
     (stroke (width 0) (type default) (color 0 0 0 0))
   )
-  (wire (pts (xy 118.11 100.33) (xy 118.11 109.22))
+  (wire (pts (xy 160.02 129.54) (xy 181.61 129.54))
     (stroke (width 0) (type default) (color 0 0 0 0))
   )
@@
     (stroke (width 0) (type default) (color 0 0 0 0))
   )
-  (wire (pts (xy 160.02 129.54) (xy 172.72 129.54))
-    (stroke (width 0) (type default) (color 0 0 0 0))
-  )
   (wire (pts (xy 175.26 82.55) (xy 177.8 82.55))
     (stroke (width 0) (type default) (color 0 0 0 0))
   )
-  (wire (pts (xy 118.11 109.22) (xy 151.13 109.22))
+  (wire (pts (xy 170.18 107.95) (xy 177.8 107.95))
     (stroke (width 0) (type default) (color 0 0 0 0))
   )
@@
     (stroke (width 0) (type default) (color 0 0 0 0))
   )
-  (wire (pts (xy 172.72 129.54) (xy 199.39 129.54))
+  (wire (pts (xy 173.99 125.73) (xy 170.18 125.73))
     (stroke (width 0) (type default) (color 0 0 0 0))
   )
@@
     (stroke (width 0) (type default) (color 0 0 0 0))
   )
-  (wire (pts (xy 193.04 105.41) (xy 193.04 116.84))
+  (wire (pts (xy 193.04 105.41) (xy 193.04 113.03))
     (stroke (width 0) (type default) (color 0 0 0 0))
   )
@@
     (stroke (width 0) (type default) (color 0 0 0 0))
   )
+  (wire (pts (xy 170.18 125.73) (xy 170.18 107.95))
+    (stroke (width 0) (type default) (color 0 0 0 0))
+  )
   (wire (pts (xy 160.02 139.7) (xy 160.02 137.16))
     (stroke (width 0) (type default) (color 0 0 0 0))
   )
-  (wire (pts (xy 160.02 109.22) (xy 160.02 110.49))
+  (wire (pts (xy 160.02 107.95) (xy 160.02 110.49))
     (stroke (width 0) (type default) (color 0 0 0 0))
   )
@@
     (stroke (width 0) (type default) (color 0 0 0 0))
   )
-  (wire (pts (xy 177.8 107.95) (xy 172.72 107.95))
-    (stroke (width 0) (type default) (color 0 0 0 0))
-  )
-  (wire (pts (xy 158.75 109.22) (xy 160.02 109.22))
+  (wire (pts (xy 157.48 107.95) (xy 160.02 107.95))
+    (stroke (width 0) (type default) (color 0 0 0 0))
+  )
+  (wire (pts (xy 118.11 107.95) (xy 149.86 107.95))
     (stroke (width 0) (type default) (color 0 0 0 0))
   )
@@
     (pin "7")
   )
-  (symbol (lib_id "Device:R") (at 193.04 120.65 0) (unit 1)
-    (in_bom yes) (on_board yes) (fields_autoplaced)
-    (property "Reference" "R?" (id 0) (at 195.58 119.3799 0)
-      (effects (font (size 1.27 1.27)) (justify left))
-    )
-    (property "Value" "R" (id 1) (at 195.58 121.9199 0)
-      (effects (font (size 1.27 1.27)) (justify left))
-    )
-    (property "Footprint" "" (id 2) (at 191.262 120.65 90)
-      (effects (font (size 1.27 1.27)) hide)
-    )
-    (property "Datasheet" "~" (id 3) (at 193.04 120.65 0)
+  (symbol (lib_id "Device:R") (at 193.04 116.84 0) (unit 1)
+    (in_bom yes) (on_board yes) (fields_autoplaced)
+    (property "Reference" "R?" (id 0) (at 195.58 115.5699 0)
+      (effects (font (size 1.27 1.27)) (justify left))
+    )
+    (property "Value" "R" (id 1) (at 195.58 118.1099 0)
+      (effects (font (size 1.27 1.27)) (justify left))
+    )
+    (property "Footprint" "" (id 2) (at 191.262 116.84 90)
+      (effects (font (size 1.27 1.27)) hide)
+    )
+    (property "Datasheet" "~" (id 3) (at 193.04 116.84 0)
       (effects (font (size 1.27 1.27)) hide)
     )
@@
     (pin "1")
   )
-  (symbol (lib_id "Device:R") (at 154.94 109.22 90) (unit 1)
-    (in_bom yes) (on_board yes) (fields_autoplaced)
-    (property "Reference" "R1" (id 0) (at 154.94 102.87 90))
-    (property "Value" "1150" (id 1) (at 154.94 105.41 90))
-    (property "Footprint" "" (id 2) (at 154.94 110.998 90)
-      (effects (font (size 1.27 1.27)) hide)
-    )
-    (property "Datasheet" "~" (id 3) (at 154.94 109.22 0)
+  (symbol (lib_id "Device:R") (at 153.67 107.95 90) (unit 1)
+    (in_bom yes) (on_board yes) (fields_autoplaced)
+    (property "Reference" "R1" (id 0) (at 153.67 101.6 90))
+    (property "Value" "1150" (id 1) (at 153.67 104.14 90))
+    (property "Footprint" "" (id 2) (at 153.67 109.728 90)
+      (effects (font (size 1.27 1.27)) hide)
+    )
+    (property "Datasheet" "~" (id 3) (at 153.67 107.95 0)
       (effects (font (size 1.27 1.27)) hide)
     )
@@
     (pin "1")
   )
-  (symbol (lib_id "Device:Q_NPN_BCE") (at 175.26 124.46 180) (unit 1)
-    (in_bom yes) (on_board yes) (fields_autoplaced)
-    (property "Reference" "Q?" (id 0) (at 170.18 123.1899 0)
-      (effects (font (size 1.27 1.27)) (justify left))
-    )
-    (property "Value" "Q_NPN_BCE" (id 1) (at 170.18 125.7299 0)
-      (effects (font (size 1.27 1.27)) (justify left))
-    )
-    (property "Footprint" "" (id 2) (at 170.18 127 0)
-      (effects (font (size 1.27 1.27)) hide)
-    )
-    (property "Datasheet" "~" (id 3) (at 175.26 124.46 0)
-      (effects (font (size 1.27 1.27)) hide)
-    )
+  (symbol (lib_id "Device:Q_NPN_BCE") (at 176.53 120.65 180) (unit 1)
+    (in_bom yes) (on_board yes) (fields_autoplaced)
+    (property "Reference" "Q?" (id 0) (at 171.45 119.3799 0)
+      (effects (font (size 1.27 1.27)) (justify left))
+    )
+    (property "Value" "Q_NPN_BCE" (id 1) (at 171.45 121.9199 0)
+      (effects (font (size 1.27 1.27)) (justify left))
+    )
+    (property "Footprint" "" (id 2) (at 171.45 123.19 0)
+      (effects (font (size 1.27 1.27)) hide)
+    )
+    (property "Datasheet" "~" (id 3) (at 176.53 120.65 0)
+      (effects (font (size 1.27 1.27)) hide)
+    )
