File: recruitment.kicad_sch (KiCad schematic)
At the start: 18 parts, among them Q1 BSN20, SW1 SW_SPST

Commit message: routing, first release
Parts:
- Rhall1, Rhall2, Rload1, Rload2, Rrelay2: footprint (none) -> Resistor_SMD:R_2816_7142Metric
- flipflop1: footprint TSSOP14_SOT402-1_NEX -> footprints:74HC74PW-Q100_118
- multiplier1: footprint N_8_ADI -> ad835:AD835AN
Changed lines of the file:
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@@
       (effects (font (size 1.524 1.524)))
     )
-    (property "Footprint" "N_8_ADI" (id 2) (at 191.77 61.214 0)
+    (property "Footprint" "ad835:AD835AN" (id 2) (at 191.77 61.214 0)
       (effects (font (size 1.524 1.524)) hide)
     )
@@
       (effects (font (size 1.27 1.27)) (justify left))
     )
-    (property "Footprint" "" (id 2) (at 158.242 59.69 90)
+    (property "Footprint" "Resistor_SMD:R_2816_7142Metric" (id 2) (at 158.242 59.69 90)
       (effects (font (size 1.27 1.27)) hide)
     )
@@
       (effects (font (size 1.524 1.524)))
     )
-    (property "Footprint" "TSSOP14_SOT402-1_NEX" (id 2) (at 191.77 120.904 0)
+    (property "Footprint" "footprints:74HC74PW-Q100_118" (id 2) (at 191.77 120.904 0)
       (effects (font (size 1.524 1.524)) hide)
     )
@@
     (property "Reference" "Rhall2" (id 0) (at 115.57 73.66 90))
     (property "Value" "10" (id 1) (at 115.57 76.2 90))
-    (property "Footprint" "" (id 2) (at 115.57 77.978 90)
+    (property "Footprint" "Resistor_SMD:R_2816_7142Metric" (id 2) (at 115.57 77.978 90)
       (effects (font (size 1.27 1.27)) hide)
     )
@@
     (property "Reference" "Rrelay2" (id 0) (at 100.33 69.85 90))
     (property "Value" "R" (id 1) (at 100.33 72.39 90))
-    (property "Footprint" "" (id 2) (at 100.33 77.978 90)
+    (property "Footprint" "Resistor_SMD:R_2816_7142Metric" (id 2) (at 100.33 77.978 90)
       (effects (font (size 1.27 1.27)) hide)
     )
@@
     (property "Reference" "Rhall1" (id 0) (at 125.73 73.66 90))
     (property "Value" "90" (id 1) (at 125.73 76.2 90))
-    (property "Footprint" "" (id 2) (at 125.73 77.978 90)
+    (property "Footprint" "Resistor_SMD:R_2816_7142Metric" (id 2) (at 125.73 77.978 90)
       (effects (font (size 1.27 1.27)) hide)
     )
@@
       (effects (font (size 1.27 1.27)) (justify left))
     )
-    (property "Footprint" "" (id 2) (at 158.242 74.93 90)
+    (property "Footprint" "Resistor_SMD:R_2816_7142Metric" (id 2) (at 158.242 74.93 90)
       (effects (font (size 1.27 1.27)) hide)
     )
@@
     )
     (path "/af630c96-ce5d-4d01-b7d8-e93460b001b7"
-      (reference "Rhall1") (unit 1) (value "90") (footprint "")
+      (reference "Rhall1") (unit 1) (value "90") (footprint "Resistor_SMD:R_2816_7142Metric")
     )
     (path "/6c7bb8ba-b4ee-4b88-9819-7838986f1407"
-      (reference "Rhall2") (unit 1) (value "10") (footprint "")
+      (reference "Rhall2") (unit 1) (value "10") (footprint "Resistor_SMD:R_2816_7142Metric")
     )
     (path "/211c7bdd-44bf-48ac-91da-f275e1d60f7b"
-      (reference "Rload1") (unit 1) (value "9900") (footprint "")
+      (reference "Rload1") (unit 1) (value "9900") (footprint "Resistor_SMD:R_2816_7142Metric")
     )
     (path "/e0acb5a4-0745-482c-903d-455adf074c4c"
-      (reference "Rload2") (unit 1) (value "100") (footprint "")
+      (reference "Rload2") (unit 1) (value "100") (footprint "Resistor_SMD:R_2816_7142Metric")
     )
     (path "/424d5b31-88ca-4b43-8316-4aec53e16753"
@@
     )
     (path "/91fc54ff-4276-41b0-a00a-1e9cd1288e91"
-      (reference "Rrelay2") (unit 1) (value "R") (footprint "")
+      (reference "Rrelay2") (unit 1) (value "R") (footprint "Resistor_SMD:R_2816_7142Metric")
     )
     (path "/5f8faae4-ef37-4fd2-bda1-cf2eb8cb91b1"
@@
     )
     (path "/371c49f2-e2b9-44ae-819d-be100bbe7a64"
-      (reference "flipflop1") (unit 1) (value "74HC74PW-Q100_118") (footprint "TSSOP14_SOT402-1_NEX")
+      (reference "flipflop1") (unit 1) (value "74HC74PW-Q100_118") (footprint "footprints:74HC74PW-Q100_118")
     )
     (path "/1fec51c3-ba3f-4cf3-9987-7bbf54f192c6"
-      (reference "multiplier1") (unit 1) (value "AD835AN") (footprint "N_8_ADI")
+      (reference "multiplier1") (unit 1) (value "AD835AN") (footprint "ad835:AD835AN")
     )
     (path "/8bd72d47-aeb7-450d-acca-ccb14d6baac1"

Commit message: check
Parts:
- Rrelay1: value R -> 10
- Rrelay2: value R -> 15
- SW1: value SW_SPST -> switch
- renumbered LoadConnector1 to LoadConnect1, SupplyConnector1 to SupplyConnect1
Connections:
- net V_pot: now also Comparator1.3 (IN+)
Changed lines of the file:
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@@
+    (stroke (width 0) (type default) (color 0 0 0 0))
+  )
+  (wire (pts (xy 165.1 102.87) (xy 171.45 102.87))
     (stroke (width 0) (type default) (color 0 0 0 0))
   )
@@
     (effects (font (size 1.27 1.27)) (justify left bottom))
   )
+  (label "V_pot" (at 165.1 102.87 0)
+    (effects (font (size 1.27 1.27)) (justify left bottom))
+  )
   (label "V_ref" (at 165.1 100.33 0)
     (effects (font (size 1.27 1.27)) (justify left bottom))
@@
       (effects (font (size 1.27 1.27)) (justify left))
     )
-    (property "Value" "R" (id 1) (at 88.9 90.1699 0)
+    (property "Value" "10" (id 1) (at 88.9 90.1699 0)
       (effects (font (size 1.27 1.27)) (justify left))
     )
@@
     (in_bom yes) (on_board yes) (fields_autoplaced)
     (property "Reference" "SW1" (id 0) (at 59.69 91.44 0))
-    (property "Value" "SW_SPST" (id 1) (at 59.69 93.98 0))
+    (property "Value" "switch" (id 1) (at 59.69 93.98 0))
     (property "Footprint" "Button_Switch_SMD:SW_DIP_SPSTx01_Slide_6.7x4.1mm_W6.73mm_P2.54mm_LowProfile_JPin" (id 2) (at 59.69 97.79 0)
       (effects (font (size 1.27 1.27)) hide)
@@
     (in_bom yes) (on_board yes) (fields_autoplaced)
     (property "Reference" "Rrelay2" (id 0) (at 100.33 69.85 90))
-    (property "Value" "R" (id 1) (at 100.33 72.39 90))
+    (property "Value" "15" (id 1) (at 100.33 72.39 90))
     (property "Footprint" "Resistor_SMD:R_2816_7142Metric" (id 2) (at 100.33 77.978 90)
       (effects (font (size 1.27 1.27)) hide)
@@
   (symbol (lib_id "Connector:Conn_01x03_Female") (at 49.53 97.79 180) (unit 1)
     (in_bom yes) (on_board yes) (fields_autoplaced)
-    (property "Reference" "SupplyConnector1" (id 0) (at 50.165 90.17 0))
+    (property "Reference" "SupplyConnect1" (id 0) (at 50.165 90.17 0))
     (property "Value" "Conn_01x03_Female" (id 1) (at 50.165 92.71 0))
     (property "Footprint" "Connector_PinHeader_2.00mm:PinHeader_1x03_P2.00mm_Vertical" (id 2) (at 49.53 97.79 0)
@@
   (symbol (lib_id "Connector:Conn_01x02_Female") (at 234.95 86.36 0) (unit 1)
     (in_bom yes) (on_board yes)
-    (property "Reference" "LoadConnector1" (id 0) (at 236.22 86.3599 0)
+    (property "Reference" "LoadConnect1" (id 0) (at 236.22 86.3599 0)
       (effects (font (size 1.27 1.27)) (justify left))
     )
@@
     )
     (path "/9ef2c0bd-0176-4f0e-b213-c48663ceb734"
-      (reference "LoadConnector1") (unit 1) (value "Conn_01x02_Female") (footprint "Connector_PinHeader_2.00mm:PinHeader_1x02_P2.00mm_Vertical")
+      (reference "LoadConnect1") (unit 1) (value "Conn_01x02_Female") (footprint "Connector_PinHeader_2.00mm:PinHeader_1x02_P2.00mm_Vertical")
     )
     (path "/f85a42e4-203a-4e25-98e4-36d444206b66"
@@
     )
     (path "/0850d44a-6bde-4886-b872-ef2fda5e1590"
-      (reference "Rrelay1") (unit 1) (value "R") (footprint "Resistor_SMD:R_2816_7142Metric")
+      (reference "Rrelay1") (unit 1) (value "10") (footprint "Resistor_SMD:R_2816_7142Metric")
     )
     (path "/91fc54ff-4276-41b0-a00a-1e9cd1288e91"
-      (reference "Rrelay2") (unit 1) (value "R") (footprint "Resistor_SMD:R_2816_7142Metric")
+      (reference "Rrelay2") (unit 1) (value "15") (footprint "Resistor_SMD:R_2816_7142Metric")
     )
     (path "/5f8faae4-ef37-4fd2-bda1-cf2eb8cb91b1"
-      (reference "SW1") (unit 1) (value "SW_SPST") (footprint "Button_Switch_SMD:SW_DIP_SPSTx01_Slide_6.7x4.1mm_W6.73mm_P2.54mm_LowProfile_JPin")
+      (reference "SW1") (unit 1) (value "switch") (footprint "Button_Switch_SMD:SW_DIP_SPSTx01_Slide_6.7x4.1mm_W6.73mm_P2.54mm_LowProfile_JPin")
     )
     (path "/9e427954-2486-4c91-89b5-6af73a073442"
-      (reference "SupplyConnector1") (unit 1) (value "Conn_01x03_Female") (footprint "Connector_PinHeader_2.00mm:PinHeader_1x03_P2.00mm_Vertical")
+      (reference "SupplyConnect1") (unit 1) (value "Conn_01x03_Female") (footprint "Connector_PinHeader_2.00mm:PinHeader_1x03_P2.00mm_Vertical")
     )
     (path "/371c49f2-e2b9-44ae-819d-be100bbe7a64"

Commit message: check R relay
Parts:
- Rrelay1: value 10 -> 30
- Rrelay2: value 15 -> 20
Changed lines of the file:
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@@
       (effects (font (size 1.27 1.27)) (justify left))
     )
-    (property "Value" "10" (id 1) (at 88.9 90.1699 0)
+    (property "Value" "30" (id 1) (at 88.9 90.1699 0)
       (effects (font (size 1.27 1.27)) (justify left))
     )
@@
     (in_bom yes) (on_board yes) (fields_autoplaced)
     (property "Reference" "Rrelay2" (id 0) (at 100.33 69.85 90))
-    (property "Value" "15" (id 1) (at 100.33 72.39 90))
+    (property "Value" "20" (id 1) (at 100.33 72.39 90))
     (property "Footprint" "Resistor_SMD:R_2816_7142Metric" (id 2) (at 100.33 77.978 90)
       (effects (font (size 1.27 1.27)) hide)
@@
     )
     (path "/0850d44a-6bde-4886-b872-ef2fda5e1590"
-      (reference "Rrelay1") (unit 1) (value "10") (footprint "Resistor_SMD:R_2816_7142Metric")
+      (reference "Rrelay1") (unit 1) (value "30") (footprint "Resistor_SMD:R_2816_7142Metric")
     )
     (path "/91fc54ff-4276-41b0-a00a-1e9cd1288e91"
-      (reference "Rrelay2") (unit 1) (value "15") (footprint "Resistor_SMD:R_2816_7142Metric")
+      (reference "Rrelay2") (unit 1) (value "20") (footprint "Resistor_SMD:R_2816_7142Metric")
     )
     (path "/5f8faae4-ef37-4fd2-bda1-cf2eb8cb91b1"

Commit message: check Rref
Parts:
- Rref1: value 4000 -> 1900
Other:
- note added: "Vref voltage divider: the Vref value must be 500*k. The multiplier inputs must be < than 1V. so V_Nhall is equal to the sensor output divided by 10 (the sensor's max output is 6.5V) and V_Nload = Vload/100. Vref must be 500/(10*100*5) * S, were S is the Hall effect sensor sensibility"
- note removed: "Vref voltage divider: the Vref value must be 500*k. The multiplier inputs must be < than 1V. so V_Nhall is equal to the sensor output divided by 10 (the sensor's max output is 6.5V) and V_Nload = Vload/100. Vref must be 500/(10*1000) * S, were S is the Hall effect sensor sensibility"
Changed lines of the file:
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@@
     (stroke (width 0) (type default) (color 0 0 0 0))
   )
-  (text "Vref voltage divider: the Vref value must be 500*k.\nThe multiplier inputs must be < than 1V. so V_Nhall is equal\nto the sensor output divided by 10 (the sensor's max output is\n6.5V) and V_Nload = Vload/100.\nVref must be 500/(10*1000) * S, were S is the Hall effect sensor\nsensibility\n"
+  (text "Vref voltage divider: the Vref value must be 500*k.\nThe multiplier inputs must be < than 1V. so V_Nhall is equal\nto the sensor output divided by 10 (the sensor's max output is\n6.5V) and V_Nload = Vload/100.\nVref must be 500/(10*100*5) * S, were S is the Hall effect sensor\nsensibility\n"
     (at 63.5 135.89 0)
     (effects (font (size 1.27 1.27)) (justify left bottom))
@@
       (effects (font (size 1.27 1.27)) (justify right))
     )
-    (property "Value" "4000" (id 1) (at 88.9 105.4099 0)
+    (property "Value" "1900" (id 1) (at 88.9 105.4099 0)
       (effects (font (size 1.27 1.27)) (justify right))
     )
@@
     )
     (path "/424d5b31-88ca-4b43-8316-4aec53e16753"
-      (reference "Rref1") (unit 1) (value "4000") (footprint "Resistor_SMD:R_2816_7142Metric")
+      (reference "Rref1") (unit 1) (value "1900") (footprint "Resistor_SMD:R_2816_7142Metric")
     )
     (path "/0688bc70-7f53-41de-a6b4-1297b52069e5"

Commit message: ses with and without vias
Other:
- note added: "relay specifics required to close the internal switch: 3V and 66.6mA"
Changed lines of the file:
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@@
+    (effects (font (size 1.27 1.27)) (justify left bottom))
+  )
+  (text "relay specifics required to close the internal switch:\n3V and 66.6mA"
+    (at 39.37 54.61 0)
     (effects (font (size 1.27 1.27)) (justify left bottom))
   )
