File: recruitment.kicad_pcb (KiCad board)
At the start: 2 copper layers, 18 parts, among them Q1 BSN20, SW1 switch

Commit message: check R relay
Parts:
- Rrelay1: value 10 -> 30
- Rrelay2: value 15 -> 20
Changed lines of the file:
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@@
       (effects (font (size 1 1) (thickness 0.15)))
     )
-    (fp_text value "15" (at 0 3.18) (layer "F.Fab")
+    (fp_text value "20" (at 0 3.18) (layer "F.Fab")
       (effects (font (size 1 1) (thickness 0.15)))
     )
@@
       (effects (font (size 1 1) (thickness 0.15)))
     )
-    (fp_text value "10" (at 0 3.18) (layer "F.Fab")
+    (fp_text value "30" (at 0 3.18) (layer "F.Fab")
       (effects (font (size 1 1) (thickness 0.15)))
     )

Commit message: check Rref
Parts:
- Rref1: value 4000 -> 1900
Changed lines of the file:
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@@
       (effects (font (size 1 1) (thickness 0.15)))
     )
-    (fp_text value "4000" (at 0 3.18) (layer "F.Fab")
+    (fp_text value "1900" (at 0 3.18) (layer "F.Fab")
       (effects (font (size 1 1) (thickness 0.15)))
     )
