File: recruitment.kicad_pcb (KiCad board)
At the start: 2 copper layers, 18 parts, among them Q1 BSN20, SW1 switch

Commit message: ses with and without vias
Routing:
- net /Vcc: track 86.2 -> 101.9 mm, vias 1 -> 0
- net /V_ff: track 48.0 -> 41.1 mm
- net GND: track 114.2 -> 120.4 mm
- net /V_ref: track 27.1 -> 21.1 mm
- net Net-(HallSensor1-Pad5): track 34.1 -> 37.2 mm
- net Net-(SW1-Pad1): track 10.4 -> 8.13 mm
- net Net-(HallSensor1-Pad3): track 20.4 -> 18.4 mm
- net Net-(HallSensor1-Pad6): track 9.56 -> 11.0 mm
- net /V_Nhall: track 27.4 -> 28.6 mm, vias 1 -> 0

Commit message: forgotten commit :)
Other:
- board outline added: 58.4 x 38.1 mm
Changed lines of the file:
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@@
     )
   )
+  (gr_rect (start 106.68 114.3) (end 165.1 76.2) (layer "Edge.Cuts") (width 0.05) (fill none))
   (segment (start 127.9858 111.7757) (end 132.0368 111.7757) (width 0.25) (layer "F.Cu") (net 2))
   (segment (start 127.7287 111.2613) (end 127.7287 111.5186) (width 0.25) (layer "F.Cu") (net 2))
